File: Kick-808.kicad_pcb (KiCad board)
At the start: 2 copper layers, 19.3 x 106.5 mm, 70 parts, among them J3 Conn_02x05_Odd_Even, Q1 BC847, Q2 BC847, Q3 BC857, Q4 BC847, Q5 BC847, Q6 BC847, Q7 BC847, SW1 SW_Push_LED, U1 TL072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

Commit message: Routing almost complete.
Parts:
- turned R12 to 0 degrees
- turned C14 to 180 degrees
- turned Q1 to 180 degrees
- turned R14 to 0 degrees
- turned R2 to 0 degrees
- turned R5 to 0 degrees
- turned R6 to 0 degrees
Routing:
- net Pulse: track 0.00 -> 86.3 mm
- net 5V: track 0.00 -> 66.3 mm, vias 0 -> 1
- net +12V: track 88.9 -> 139.5 mm, vias 2 -> 9
- net Net-(C10-Pad1): track 0.00 -> 48.0 mm, vias 0 -> 2
- net Net-(Accent1-PadT): track 0.00 -> 40.5 mm, vias 0 -> 1
- net GND: track 0.00 -> 38.2 mm, vias 0 -> 27
- net Net-(C5-Pad2): track 0.00 -> 37.7 mm, vias 0 -> 2
- net -12V: track 40.7 -> 77.3 mm, vias 2 -> 3
- net Net-(Output1-PadT): track 0.00 -> 34.2 mm
- net Net-(Decay1-Pad1): track 0.00 -> 31.6 mm
- net Net-(C13-Pad2): track 0.00 -> 27.8 mm, vias 0 -> 2
- net Net-(Q3-Pad2): track 0.00 -> 25.6 mm
- net Net-(C9-Pad2): track 0.00 -> 23.6 mm
- net Net-(Mod1-Pad2): track 0.00 -> 22.6 mm, vias 0 -> 1
- net Net-(C11-Pad1): track 0.00 -> 19.6 mm
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- added copper zone on B.Cu, net GND

Commit message: Routing completed.
Parts:
- moved C15 2.84 mm to (123.6, 101.5), turned to 180 degrees
- moved R4 2.79 mm to (123.6, 104.4)
Routing:
- net +12V: track 139.5 -> 142.3 mm, vias 9 -> 10
- net Net-(Accent1-PadT): track 40.5 -> 38.0 mm
- net -12V: track 77.3 -> 79.0 mm, vias 3 -> 4
- net Net-(C11-Pad1): track 19.6 -> 20.3 mm

Commit message: Routing adjustments.
Parts:
- moved R27 2.79 mm to (130.6, 84.8), turned to 180 degrees
- moved R29 2.79 mm to (130.6, 82.0)
Connections:
- Decay1 pad : (no net) -> GND
- Mod1 pad : (no net) -> GND
- Mod2 pad : (no net) -> GND
- Tone1 pad : (no net) -> GND
Routing:
- net Net-(C5-Pad2): track 37.7 -> 44.8 mm
- net Net-(R27-Pad1): track 6.46 -> 3.84 mm
- net Net-(Mod1-Pad2): track 22.6 -> 21.3 mm
- net Pulse: track 86.3 -> 87.2 mm
- net Net-(Decay1-Pad1): track 31.6 -> 32.5 mm
- net -12V: track 79.0 -> 78.4 mm
- net GND: vias 27 -> 18
