File: Kick-808.kicad_pcb (KiCad board)
At the start: 2 copper layers, 19.3 x 106.5 mm, 70 parts, among them J3 Conn_02x05_Odd_Even, Q1 BC847, Q2 BC847, Q3 BC857, Q4 BC847, Q5 BC847, Q6 BC847, Q7 BC847, SW1 SW_Push_LED, U1 TL072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

Commit message: Branding.
Other:
- board text added: "+12V"
- board text added: "-12V"
- board text added: "Kick Clone"
- board text added: "Marangisto 2020"
- board text added: "TR-808"
Changed lines of the file:
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@@
   (general
     (thickness 1.6)
-    (drawings 38)
+    (drawings 45)
     (tracks 500)
     (zones 0)
@@
     )
   )
+  (gr_line (start 122.301 78.613) (end 122.301 93.218) (layer B.SilkS) (width 0.15))
+  (gr_text "Kick Clone" (at 123.571 85.979 90) (layer B.SilkS)
+    (effects (font (size 1 1.8) (thickness 0.2)) (justify mirror))
+  )
+  (gr_text "TR-808\n" (at 120.015 86.106 90) (layer B.SilkS)
+    (effects (font (size 3 2.5) (thickness 0.3)) (justify mirror))
+  )
+  (gr_text "Marangisto 2020" (at 127.254 152.908) (layer B.SilkS)
+    (effects (font (size 1 1) (thickness 0.15)) (justify mirror))
+  )
+  (gr_text -12V (at 135.255 143.637 90) (layer B.SilkS)
+    (effects (font (size 1 1) (thickness 0.15)) (justify mirror))
+  )
+  (gr_text +12V (at 119.634 143.637 90) (layer B.SilkS)
+    (effects (font (size 1 1) (thickness 0.15)) (justify mirror))
+  )
+  (gr_line (start 134.112 141.478) (end 134.112 146.177) (layer B.SilkS) (width 0.4))
   (gr_circle (center 127 52.349999) (end 129.8 52.349999) (layer Dwgs.User) (width 0.2))
   (gr_circle (center 127.022308 125.850024) (end 130.072308 125.850024) (layer Dwgs.User) (width 0.2))

Commit message: Generated gerbers.
Other:
- board text added: "Rev A"
Changed lines of the file:
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@@
   (general
     (thickness 1.6)
-    (drawings 45)
+    (drawings 46)
     (tracks 500)
     (zones 0)
@@
       (viasonmask false)
       (mode 1)
-      (useauxorigin false)
+      (useauxorigin true)
       (hpglpennumber 1)
       (hpglpenspeed 20)
@@
       (outputformat 1)
       (mirror false)
-      (drillshape 1)
+      (drillshape 0)
       (scaleselection 1)
-      (outputdirectory ""))
+      (outputdirectory "Gerber"))
   )
   (net 0 "")
@@
     )
   )
+  (gr_text "Rev A" (at 132.588 60.071) (layer B.SilkS)
+    (effects (font (size 1 1) (thickness 0.15)) (justify mirror))
+  )
   (gr_line (start 122.301 78.613) (end 122.301 93.218) (layer B.SilkS) (width 0.15))
